File: maestro.sch (KiCad schematic (older format))
At the start: 26 parts

Commit message: Release v2
Parts:
- removed C? (x2): 1n, Capacitors_SMD:C_0603_HandSoldering, symbol Device:C
- removed FB?: Ferrite_Bead_Small, symbol Device:Ferrite_Bead_Small
- removed J?: Conn_01x04_Male, symbol Connector:Conn_01x04_Male
- removed R?: 10m, Resistors_SMD:R_0603_HandSoldering, symbol Device:R_Shunt
- removed R? (x2): 100, Resistors_SMD:R_0603_HandSoldering, symbol Device:R
- removed R? (x4): 100k, Resistors_SMD:R_0603_HandSoldering, symbol Device:R
- removed U? (x3): MCP6561-OT, Package_TO_SOT_SMD:SOT-23-5, symbol Comparator:MCP6561-OT
- added C3: 100n, Capacitor_SMD:C_0603_1608Metric_Pad1.08x0.95mm_HandSolder, symbol Device:C
- added D1, D2: LED, LEDs:LED_0603_HandSoldering, symbol Device:LED
- added J3: Conn_01x07_Female, Pin_Headers:Pin_Header_Straight_1x09_Pitch2.54mm, symbol Connector:Conn_01x09_Male
- added J4: Conn_01x03_Female, Pin_Headers:Pin_Header_Straight_1x03_Pitch2.54mm, symbol Connector:Conn_01x03_Male
- added R1, R11, R13, R14, R15: 2k2, Resistor_SMD:R_0603_1608Metric_Pad0.98x0.95mm_HandSolder, symbol Device:R
- added R2: 10m, Resistors_SMD:R_1206_HandSoldering, symbol Device:R
- added R5, R8: 15k, Resistor_SMD:R_0603_1608Metric_Pad0.98x0.95mm_HandSolder, symbol Device:R
- added U2: LM339, Package_SO:SOIC-14_3.9x8.7mm_P1.27mm, symbol Comparator:LM339
- C1, C2: renamed from C?; footprint Capacitors_SMD:C_0603_HandSoldering -> Capacitor_SMD:C_0603_1608Metric_Pad1.08x0.95mm_HandSolder
- FB2: renamed from FB?; footprint (none) -> Inductors_SMD:L_0603_HandSoldering
- J1: renamed from J?; footprint (none) -> proj_footprints:HIROSE_CX60-24S-UNIT
- J2: renamed from J?; footprint (none) -> proj_footprints:USB_C_Receptable_JAE_DX07S016JA1
- R10, R9: renamed from R?; value 1Meg -> 220k; footprint Resistors_SMD:R_0603_HandSoldering -> Resistor_SMD:R_0603_1608Metric_Pad0.98x0.95mm_HandSolder
- R3, R4: renamed from R?; value 1k -> 2k2; footprint Resistors_SMD:R_0603_HandSoldering -> Resistor_SMD:R_0603_1608Metric_Pad0.98x0.95mm_HandSolder
- R6: renamed from R?; value 100k -> 15k; footprint Resistors_SMD:R_0603_HandSoldering -> Resistor_SMD:R_0603_1608Metric_Pad0.98x0.95mm_HandSolder
- R7: renamed from R?; value 100k -> 2k2; footprint Resistors_SMD:R_0603_HandSoldering -> Resistor_SMD:R_0603_1608Metric_Pad0.98x0.95mm_HandSolder
- U1: renamed from U?; footprint Package_TO_SOT_SMD:SOT-89-3 -> TO_SOT_Packages_SMD:SOT-89-3_Handsoldering
Connections:
- net labels added: CC1_, CC2_, D+, D-, HV, HV_, SBU1, SBU2, SHIELD, VBUS1, VBUS2, VREF
- net labels removed: DM, DP
- wire segments 66 -> 70
Other:
- moved on the sheet: C1, C2, FB2, J1, J2, R10, R3, R4, R6, R7, R9, U1
